Commit message: update config

File: description/camera.xacro (robot description, xacro)
@@ -4,5 +4,5 @@
         <parent link="chassis"/>
         <child link="camera_link"/>
-        <origin xyz="0.276 0 0.181" rpy="0 0 0"/>
+        <origin xyz="0.350 0 0.181" rpy="0 0 0"/>
     </joint>
     <link name="camera_link">
